File: PCB/Open_80017a.kicad_sch (KiCad schematic)
At the start: 52 parts, among them J1 Conn_01x12, Q1 MMDT3906, Q2 ZVP1320F, Q3 ZVP1320F, Q4 ZVP1320F, Q5 ZVP1320F, U1 LM13700, U2 LM13700, U3 LM13700, U4 TL072

Commit message: fix .prl
Parts:
- J1: now not fitted
Changed lines of the file:
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@@
 		(in_bom yes)
 		(on_board yes)
-		(dnp no)
+		(dnp yes)
 		(fields_autoplaced yes)
 		(property "Reference" "J1"
